File: pcb/pwr.kicad_sch (KiCad schematic)
At the start: 6 parts, among them U1 GW1N-6&9_QN48

Commit message: pcb: schemat rev. A
Parts:
- removed C1, C2, C3, C4, C5: 100n, Capacitor_SMD:C_0603_1608Metric, symbol Device:C
- removed U1: GW1N-6&9_QN48, Package_DFN_QFN:QFN-48-1EP_6x6mm_P0.4mm_EP4.2x4.2mm_ThermalVias, symbol gowin_fpga:GW1N-6&9_QN48
