File: pcb/ext_io.kicad_sch (KiCad schematic)
At the start: 11 parts, among them J2 TC2050, U1 GW1N-6&9_QN48

Commit message: pcb: schemat rev. A
Parts:
- added C1, C13, C19, C2, C3, C4, C5: 100n, Capacitor_SMD:C_0603_1608Metric, symbol Device:C
- added C14, C15, C16, C17, C18: 10u, Capacitor_SMD:C_0603_1608Metric, symbol Device:C
- added D1: SMF3.3A, Diode_SMD:D_SOD-123F, symbol Device:D_Zener
- added J3: Conn_02x10_Odd_Even, Connector_PinHeader_1.27mm:PinHeader_2x10_P1.27mm_Vertical, symbol Connector_Generic:Conn_02x10_Odd_Even
- added R13: 4.7k, Resistor_SMD:R_0603_1608Metric, symbol Device:R
- added unit 5 of U1
- R2: value 10k -> 1k
Connections:
- net +3V3: now also C1.1, C13.1, C14.2, C15.2, C16.2, C17.2, C18.2, C19.1, C2.1, C3.1, C4.1, C5.1, D1.1 (K), J3.1 (Pin_1), J3.2 (Pin_2), U1.1 (VCCO0/VCCO3), U1.12 (VCC[2]), U1.25 (VCCO1/VCCO2), U1.36 (VCCX), U1.37 (VCC[2])
- net GND: now also C1.2, C13.2, C14.1, C15.1, C16.1, C17.1, C18.1, C19.2, C2.2, C3.2, C4.2, C5.2, D1.2 (A), J3.15 (Pin_15), J3.19 (Pin_19), J3.20 (Pin_20), J3.3 (Pin_3), J3.5 (Pin_5), R13.2, U1.2 (VSS[2]), U1.26 (VSS[2])
- net HOST_IRQ_N: now also J3.17 (Pin_17)
- net HOST_RST_N: now also J3.18 (Pin_18)
- net TCK: now also R13.1
- net XSPI_CS_N: now also J3.6 (Pin_6)
- net XSPI_DQS: now also J3.16 (Pin_16)
- net XSPI_IO0: now also J3.7 (Pin_7)
- net XSPI_IO1: now also J3.8 (Pin_8)
- net XSPI_IO2: now also J3.9 (Pin_9)
- net XSPI_IO3: now also J3.10 (Pin_10)
- net XSPI_IO4: now also J3.11 (Pin_11)
- net XSPI_IO5: now also J3.12 (Pin_12)
- net XSPI_IO6: now also J3.13 (Pin_13)
- net XSPI_IO7: now also J3.14 (Pin_14)
- net XSPI_SCLK: now also J3.4 (Pin_4)
Other:
- moved on the sheet: JP2, R3, R4, R6, R7

Commit message: pcb: rozmieszczenie i czesc routingu, odwrocona para RD, reguly i klasy sieci
Parts:
- added JP3: SolderJumper_2_Open, Jumper:SolderJumper-2_P1.3mm_Open_TrianglePad1.0x1.5mm, symbol Jumper:SolderJumper_2_Open
- added R16: 10k, Resistor_SMD:R_0603_1608Metric, symbol Device:R
Connections:
- net +3V3: now also R16.1
- net GND: now also JP3.1 (A)
- net MODE_SEL: now reaches U1.10 (IOL15A/GCLKT_6)
- net MODE_SEL: now also JP3.2 (B), R16.2
- no-connect marks 1 -> 0

Commit message: pcb: routing par LVDS, zasilania i magistrali xSPI
Connections:
- net GND renamed EPAD
- net EPAD: now also U1.49 (EPAD)
Changed lines of the file:
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@@
 		(pin "37"
 		)
+		(pin "49"
+		)
 		(instances
 			(project "SFP_xSPI_Bridge"
@@
 		(fields_autoplaced yes)
 		(property "Reference" "U1"
-			(at 175.26 63.4999 0)
+			(at 172.72 54.6099 0)
 			(show_name no)
 			(do_not_autoplace no)
@@
 		)
 		(property "Value" "GW1N-6&9_QN48"
-			(at 175.26 66.0399 0)
+			(at 172.72 57.1499 0)
 			(show_name no)
 			(do_not_autoplace no)
@@
 		(pin "37"
 		)
+		(pin "49"
+		)
 		(instances
 			(project "SFP_xSPI_Bridge"
@@
 		(fields_autoplaced yes)
 		(property "Reference" "U1"
-			(at 205.74 123.1899 0)
+			(at 187.96 113.0299 0)
 			(show_name no)
 			(do_not_autoplace no)
@@
 		)
 		(property "Value" "GW1N-6&9_QN48"
-			(at 205.74 125.7299 0)
+			(at 187.96 115.5699 0)
 			(show_name no)
 			(do_not_autoplace no)
@@
 		(pin "37"
 		)
+		(pin "49"
+		)
 		(instances

Commit message: pcb: rev. A - obrys, strefy, pull-up SFP_TX_DIS, via stitching, usuniete puste arkusze; pliki produkcyjne: gerbery (zip), PDF schematu i PCB, iBOM, rendery 3D
Other:
- company: (none) -> bartkepl
- title: (none) -> SFP_xSPI_Bridge
Changed lines of the file:
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@@
 	(generator_version "10.0")
 	(paper "A4")
+	(title_block
+		(title "SFP_xSPI_Bridge")
+		(date "2026-10-09")
+		(rev "A")
+		(company "bartkepl")
+	)
 	(junction
 		(at 90.17 181.61)
